Commit message: fix gpio config

File: kuka_rsi_driver/config/gpio_config.xacro (robot description, xacro)
@@ -1,11 +1,11 @@
 <?xml version="1.0"?>
 <robot xmlns:xacro="http://www.ros.org/wiki/xacro">
-  <xacro:macro name="gpio_config">
-    <gpio name="gpio">
-      <command_interface name="01" data_type="BOOL">
+  <xacro:macro name="gpio_config" params="prefix">
+    <gpio name="${prefix}gpio">
+      <command_interface name="${prefix}_command_01" data_type="BOOL">
         <limits enable="false"/>
         <param name="initial_value">0.0</param>
       </command_interface>
-      <state_interface name="01" data_type="BOOL">
+      <state_interface name="${prefix}_state_01" data_type="BOOL">
         <limits enable="false"/>
         <param name="initial_value">0.0</param>
